File: PCB/controller/controller.kicad_pcb (KiCad board)
At the start: 2 copper layers, 120 x 120 mm, 14 parts, among them J1 Connector2, U1 Switch1, U2 Loline_d_32, U3 L7805, U4 Kp, U5 Ki, U6 Kd, U7 LCD

Commit message: Update Gerber Files
Other:
- board text added: "BAT"
- board text added: "GND"
Changed lines of the file:
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@@
       (outputformat 1)
       (mirror false)
-      (drillshape 1)
+      (drillshape 0)
       (scaleselection 1)
-      (outputdirectory "")
+      (outputdirectory "gerber/")
     )
   )
@@
     (effects (font (size 1.5 1.5) (thickness 0.2)))
   )
+  (gr_text "GND" (at 81.57 29.81) (layer "F.SilkS")
+    (effects (font (size 1 1) (thickness 0.15)))
+  )
   (gr_text "I\n" (at 130.12 123.83) (layer "F.SilkS")
     (effects (font (size 1.5 1.5) (thickness 0.2)))
@@
   (gr_text "D" (at 162.63 123.59) (layer "F.SilkS")
     (effects (font (size 1.5 1.5) (thickness 0.2)))
+  )
+  (gr_text "BAT" (at 81.51 26.62) (layer "F.SilkS")
+    (effects (font (size 1 1) (thickness 0.15)))
   )
   (segment (start 98.58 38.03) (end 99.98 39.43) (width 1) (layer "F.Cu") (net 1))
@@
   (segment (start 112.22 27.03) (end 118.01 27.03) (width 1) (layer "F.Cu") (net 3))
   (via (at 140.77 84.25) (size 0.8) (drill 0.4) (layers "F.Cu" "B.Cu") (net 3))
-  (segment (start 131.21 114.56) (end 134.84 110.93) (width 1) (layer "B.Cu") (net 3))
   (segment (start 95.94 119.88) (end 101.26 114.56) (width 1) (layer "B.Cu") (net 3))
+  (segment (start 131.21 114.56) (end 140.77 105) (width 1) (layer "B.Cu") (net 3))
   (segment (start 101.26 114.56) (end 131.21 114.56) (width 1) (layer "B.Cu") (net 3))
   (segment (start 125.96 119.81) (end 131.21 114.56) (width 1) (layer "B.Cu") (net 3))
-  (segment (start 140.77 105) (end 134.84 110.93) (width 1) (layer "B.Cu") (net 3))
   (segment (start 152.34 114.56) (end 157.49 119.71) (width 1) (layer "B.Cu") (net 3))
   (segment (start 124.83 119.81) (end 125.96 119.81) (width 1) (layer "B.Cu") (net 3))
